File: vlvts/pcb/top/vlvts_top/leds.kicad_sch (KiCad schematic)
At the start: 49 parts, among them Q1 YJL2305A-YAN, Q2 YJL2305A-YAN, Q3 YJL2305A-YAN, U5 SCT2024CSSG

Commit message: vlvts: new pcb
Parts:
- U5: footprint Package_SO:SOP-24_7.5x15.4mm_P1.27mm -> Package_SO:SSOP-24_3.9x8.7mm_P0.635mm
Changed lines of the file:
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@@
 (kicad_sch
-	(version 20231120)
+	(version 20250114)
 	(generator "eeschema")
-	(generator_version "8.0")
+	(generator_version "9.0")
 	(paper "A4")
 	(junction
@@
 			)
 		)
-		(property "Footprint" "Package_SO:SOP-24_7.5x15.4mm_P1.27mm"
+		(property "Footprint" "Package_SO:SSOP-24_3.9x8.7mm_P0.635mm"
 			(at 88.9 76.2 0)
 			(effects
